File: hardware/board/ember.kicad_sch (KiCad schematic)
At the start: 74 parts, among them Q1 IRFB3207PBF, SW1 SW_Push, SW2 SW_Push, U1 TPS25730D, U10 W25Q256JVFIQT, U11 NT3H2111W0FHKH, U2 TPD6S300A, U3 STM32WB55REVx, U4 TLP183(GRH-TPL,E(T, U5 LM22676MR-ADJ, U6 MAX6675ISA+T, U7 SZYY0402Y_C434450, U8 INA226, U9 TMP119AIYBGR, X1 XL7EL89CKI-111YLC-32M, X2 X201232768KJD2SI

Commit message: peripherals and pinout
Parts:
- removed U10: W25Q256JVFIQT, lcsc:SOIC-16_L10.3-W7.5-P1.27-LS10.3-BL, symbol lcsc:W25Q256JVFIQT
- removed U7: SZYY0402Y_C434450, lcsc:LED0402-FD_YELLOW, symbol lcsc:SZYY0402Y_C434450
- added C30, C31: 100nF, Capacitor_SMD:C_0402_1005Metric, symbol Device:C
- added C32: 220nF, Capacitor_SMD:C_0603_1608Metric, symbol Device:C
- added C33: 22uF, Capacitor_SMD:CP_Elec_6.3x5.4, symbol Device:C_Polarized
- added C34: 6.8uF, Capacitor_SMD:C_0805_2012Metric, symbol Device:C
- added C35: 10nF, symbol Device:C
- added C36: 120uF, Capacitor_SMD:CP_Elec_6.3x7.7, symbol Device:C_Polarized
- added D2: 1N4148W, Diode_SMD:D_SOD-123, symbol Diode:1N4148W
- added D3: SS56, lcsc:SMA_L4.3-W2.6-LS5.2-RD, symbol lcsc:SS56
- added L2: 25X48MM_NFC_ANTENNA, lcsc:25X48MM_NFC_ANTENNA, symbol Device:L
- added L3: FXL0650-8R2-M, lcsc:IND-SMD_L7.0-W6.6_FXL0650, symbol lcsc:FXL0650-8R2-M
- added Q2: 2SC1815_C727146, lcsc:SOT-23-3_L2.9-W1.3-P1.90-LS2.4-BR, symbol lcsc:2SC1815_C727146
- added R21: HOLLR2512-3W-2MR-1%, lcsc:RES-SMD_L6.4-W3.2-1, symbol lcsc:HOLLR2512-3W-2MR-1%
- added R22, R23, R25: 4.7K, Resistor_SMD:R_0201_0603Metric, symbol Device:R
- added R24: 470, Resistor_SMD:R_0201_0603Metric, symbol Device:R
- added R26: 1.54K, symbol Device:R
- added R27: 976, symbol Device:R
- added U10: W25Q256JVEIQTR, lcsc:WSON-8_L8.0-W6.10-P1.27-BL-EP, symbol lcsc:W25Q256JVEIQTR
- R12: value 10K -> 4.7K
- R17: value 150 -> 470K; footprint Resistor_SMD:R_0201_0603Metric -> (none)
Connections:
- net LED is gone; now on an unnamed net: R17.2
- net LED_GOOD is gone; now on net FIELD_DETECT: U3.26 (PC5)
- net LED_WARNING is gone; now on net TEMP_ALERT: U3.27 (PB2)
- net VIN_3V3 is gone; now on net +3.3V: C8.1
- net +3.3V: now also BUZZER1.1, U11.6 (VCC), U11.7 (VOUT), C31.1, C32.2, C36.1, D2.1 (K), L3.2, R22.1, R23.1, R25.1, R26.1, U10.8 (VCC)
- net BUTTON: now also U3.10 (PC1); no longer U3.25 (PC4)
- net CAP_MIS: now also U3.65 (PB5); no longer U3.10 (PC1)
- net ENC_A: now also U3.9 (PC0); no longer U3.23 (PA8)
- net ENC_B: now also U3.11 (PC2); no longer U3.24 (PA9)
- net FAULT_IN: now also U3.63 (PB3); no longer U3.12 (PC3)
- net GND: now also U11.2 (VSS), U5.6 (GND), U5.9 (EP), U8.1 (A1), U8.2 (A0), U8.7 (GND), U9.B2 (GND), U9.C1 (ADD0), C30.2, C31.2, C32.1, C33.2, C34.2, C36.2, D3.2 (A), Q2.2 (E), R27.2, U10.4 (GND)
- net I2C_SCL: now also U11.3 (SCL), U9.A2 (SCL)
- net I2C_SDA: now also U11.5 (SDA), U9.A1 (SDA)
- net PPHV: now also R17.1, U5.7 (VIN), C33.1, C34.1
- net PT: now also U3.12 (PC3); no longer U3.9 (PC0)
- net SINK_EN: now also U3.64 (PB4); no longer U3.11 (PC2)
- net TEMP_CS: now also U3.46 (PB12); no longer U3.19 (PA4)
- net TEMP_MISO: now also U3.48 (PB14); no longer U3.21 (PA6)
- net TEMP_SCK: now also U3.47 (PB13); no longer U3.20 (PA5)
- net at BUZZER1.2: now also D2.2 (A), Q2.3 (C)
- net at U5.1 (BOOT): now also C35.1
- net at U5.4 (FB): now also R26.2, R27.1
- net at U5.8 (SW): now also C35.2, D3.1 (K), L3.1
- net at U8.10 (Vin+): now also R21.1
- net CURRENT_ALERT: now reaches U8.3 (~{Alert})
- net CURRENT_ALERT: now also U3.2 (PC13), R22.2
- net POWER_SDA: now reaches U8.4 (SDA)
- net POWER_SDA: now also R14.2, U1.8 (I2Ct_SDA), U3.67 (PB7)
- net POWER_SCL: now reaches U8.5 (SCL)
- net POWER_SCL: now also R13.2, U1.9 (I2Ct_SCL), U3.66 (PB6)
- net at U8.6 (VS): now also C30.1
- net at U8.8 (Vbus): now also U8.9 (Vin-), R21.2
- net FLASH_CS: now reaches U3.17 (PA2)
- net FLASH_CS: now also U10.1 (~{CS})
- net FLASH_CLK: now reaches U3.18 (PA3)
- net FLASH_CLK: now also U10.6 (CLK)
- net FLASH_IO2: now reaches U3.22 (PA7)
- net FLASH_IO2: now also U10.3 (WP#(IO2))
- net LED_BLUE: now reaches U3.38 (PB0)
- net LED_GREEN: now reaches U3.39 (PB1)
- net LED_RED: now reaches U3.40 (PE4)
- net LED_COOLING: now reaches U3.58 (PC10)
- net LED_REFLOW: now reaches U3.59 (PC11)
- net LED_SOAK: now reaches U3.60 (PC12)
- net LED_PREHEAT: now reaches U3.61 (PD0)
- net LED_PD: now reaches U3.62 (PD1)
- net TEMP_ALERT: now reaches U9.C2 (ALERT)
- net TEMP_ALERT: now also R23.2
- net at U11.1 (LA): now also L2.1
- net FIELD_DETECT: now reaches U11.4 (FD)
- net FIELD_DETECT: now also R25.2
- net at U11.8 (LB): now also L2.2
- removed net PD_SCL: R13.2, U1.9 (I2Ct_SCL), U3.6 (PB8)
- removed net PD_SDA: R14.2, U1.8 (I2Ct_SDA), U3.7 (PB9)
- new net: Q2.1 (B), R24.2
- new net BUZZER: R24.1, U3.23 (PA8)
- new net FLASH_IO0: U10.5 (DI(IO0)), U3.7 (PB9)
- new net FLASH_IO1: U10.2 (DO(IO1)), U3.6 (PB8)
- new net FLASH_IO3: U10.7 (HOLD#orRESET#(IO3)), U3.21 (PA6)
Other:
- moved on the sheet: AE1, BUZZER1, C10, C13, C14, C15, C16, C17, C18, C19, C20, C21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

Commit message: finished schematic and started PCB
Parts:
- added Brd1: SSD1306, SSD1306:128x64OLED, symbol SSD1306-128x64_OLED:SSD1306
- added C19, C30, C33, C35, C38: 100nF, Capacitor_SMD:C_0402_1005Metric, symbol Device:C
- added D10, D11, D12, D5, D6, D7, D8, D9: LED, LED_SMD:LED_0603_1608Metric, symbol Device:LED
- added D2: SS56, lcsc:SMA_L4.3-W2.6-LS5.2-RD, symbol lcsc:SS56
- added D3: 15V, lcsc:SOD-323_L1.7-W1.3-LS2.6-RD, symbol lcsc:BZT52C15S_C19077448
- added L3: 10nH, Inductor_SMD:L_0603_1608Metric, symbol Device:L
- added R21, R22: 1K, Resistor_SMD:R_0402_1005Metric, symbol Device:R
- added R24, R29, R30, R31, R32, R33, R34, R35, R36: 100, Resistor_SMD:R_0402_1005Metric, symbol Device:R
- added R37, R38: 10K, Resistor_SMD:R_0402_1005Metric, symbol Device:R
- added R39: 400, Resistor_SMD:R_0402_1005Metric, symbol Device:R
- added SW1: EC11E18244A5, lcsc:SW-TH_EC11E18244A5, symbol lcsc:EC11E18244A5
- added U11, U4: DB128L-5.08-2P-BK-S, lcsc:CONN-TH_2P-P5.08_DB128L-5.08-2P-BK-S, symbol lcsc:DB128L-5.08-2P-BK-S
- added U12: MAX31865xTP, Package_DFN_QFN:TQFN-20-1EP_5x5mm_P0.65mm_EP3.25x3.25mm, symbol Sensor_Temperature:MAX31865xTP
- added U14: DB128L-5.08-3P-BK-S, lcsc:CONN-TH_3P-P5.08_DB128L-5.08-3P-BK-S, symbol lcsc:DB128L-5.08-3P-BK-S
- C1, C2: footprint (none) -> Capacitor_SMD:C_0805_2012Metric
- C10: renamed from C8; footprint (none) -> Capacitor_SMD:C_0402_1005Metric
- C11: renamed from C9; footprint (none) -> Capacitor_SMD:C_0603_1608Metric
- C12: renamed from C35; footprint (none) -> Capacitor_SMD:C_0402_1005Metric
- C13: renamed from C10; footprint (none) -> Capacitor_SMD:C_0603_1608Metric
- C18: renamed from C29; footprint Capacitor_SMD:C_0402_1005Metric -> Capacitor_SMD:C_0603_1608Metric
- C26: renamed from C22; footprint Capacitor_SMD:C_0402_1005Metric -> Capacitor_SMD:C_0603_1608Metric
- C27: renamed from C24; footprint Capacitor_SMD:C_0402_1005Metric -> Capacitor_SMD:C_0603_1608Metric
- C31: renamed from C16; footprint Capacitor_SMD:C_0402_1005Metric -> Capacitor_SMD:C_0603_1608Metric
- C36: renamed from C27; footprint Capacitor_SMD:C_0402_1005Metric -> Capacitor_SMD:C_0603_1608Metric
- C37: renamed from C17; footprint Capacitor_SMD:C_0201_0603Metric -> Capacitor_SMD:C_0402_1005Metric
- C39: renamed from C18; footprint Capacitor_SMD:C_0201_0603Metric -> Capacitor_SMD:C_0402_1005Metric
- C4: renamed from C3; footprint (none) -> Capacitor_SMD:C_0603_1608Metric
- C40: renamed from C19; footprint Capacitor_SMD:C_0201_0603Metric -> Capacitor_SMD:C_0402_1005Metric
- C41: renamed from C20; footprint Capacitor_SMD:C_0201_0603Metric -> Capacitor_SMD:C_0402_1005Metric
- C5: renamed from C4; footprint (none) -> Capacitor_SMD:C_0805_2012Metric
- C6: renamed from C34; footprint Capacitor_SMD:C_0805_2012Metric -> Capacitor_SMD:C_0603_1608Metric
- C7: renamed from C5; footprint (none) -> Capacitor_SMD:C_0603_1608Metric
- C8: renamed from C6; footprint (none) -> Capacitor_SMD:C_0402_1005Metric
- C9: renamed from C7; footprint (none) -> Capacitor_SMD:C_0603_1608Metric
- D13: renamed from D1; footprint PCM_Diode_SMD_AKL:D_SOD-323_TVS -> Diode_SMD:D_SOD-323
- R1, R4: footprint (none) -> Resistor_SMD:R_0603_1608Metric
- R10: renamed from R9; footprint (none) -> Resistor_SMD:R_0402_1005Metric
- R11: renamed from R12; footprint (none) -> Resistor_SMD:R_0402_1005Metric
- R12: renamed from R10; footprint (none) -> Resistor_SMD:R_0603_1608Metric
- R13: renamed from R11; footprint (none) -> Resistor_SMD:R_0402_1005Metric
- R14: renamed from R13; footprint (none) -> Resistor_SMD:R_0402_1005Metric
- R15: renamed from R27; footprint (none) -> Resistor_SMD:R_0402_1005Metric
- R16: renamed from R14; footprint (none) -> Resistor_SMD:R_0402_1005Metric
- R17: renamed from R26; footprint (none) -> Resistor_SMD:R_0402_1005Metric
- R19: renamed from R23; footprint Resistor_SMD:R_0201_0603Metric -> Resistor_SMD:R_0402_1005Metric
- R2, R3: footprint (none) -> Resistor_SMD:R_0402_1005Metric
- R23: renamed from R22; footprint Resistor_SMD:R_0201_0603Metric -> Resistor_SMD:R_0402_1005Metric
- R25: footprint Resistor_SMD:R_0201_0603Metric -> Resistor_SMD:R_0402_1005Metric
- R26: renamed from R24; footprint Resistor_SMD:R_0201_0603Metric -> Resistor_SMD:R_0402_1005Metric
- R27: renamed from R19; footprint Resistor_SMD:R_0201_0603Metric -> Resistor_SMD:R_0402_1005Metric
- R28: renamed from R20; footprint Resistor_SMD:R_0201_0603Metric -> Resistor_SMD:R_0402_1005Metric
- R40: renamed from R16; footprint Resistor_SMD:R_0201_0603Metric -> Resistor_SMD:R_0402_1005Metric
- R41: renamed from R18; footprint Resistor_SMD:R_0201_0603Metric -> Resistor_SMD:R_0402_1005Metric
- R5: renamed from R17; footprint (none) -> Resistor_SMD:R_0603_1608Metric
- R6: renamed from R5; footprint (none) -> Resistor_SMD:R_0603_1608Metric
- R7: renamed from R6; footprint (none) -> Resistor_SMD:R_0402_1005Metric
- R8: renamed from R7; footprint (none) -> Resistor_SMD:R_0402_1005Metric
- R9: renamed from R8; footprint (none) -> Resistor_SMD:R_0402_1005Metric
- renumbered C36 to C14, C11 to C15, C30 to C16, C12 to C17, C31 to C20, C32 to C21, C21 to C22, C25 to C24, C13 to C25, C14 to C28, C15 to C29, C33 to C3, C26 to C32, C28 to C34, D3 to D1, D2 to D4, L3 to L1, L1 to L2, L2 to L4, R21 to R18, R15 to R20, SW1 to SW2, SW2 to SW3, U11 to U10, U6 to U13, U5 to U2, U2 to U3, U8 to U5, U9 to U6, U4 to U7, U10 to U8, U3 to U9
Connections:
- net TEMP_CS is gone; now on net THERMO_CS: U9.46 (PB12)
- net TEMP_MISO is gone; now on net THERMO_MISO: U9.48 (PB14)
- net TEMP_SCK is gone; now on net THERMO_SCK: U9.47 (PB13)
- net +3.3V: now also U13.4 (VCC), U6.B1 (V+), Brd1.2 (VCC), C19.1, C30.1, C33.1, C35.1, R29.2, R30.2, R31.2, R32.2, R33.2, R34.2, R35.2, R36.2, R37.1, R38.1, U12.19 (DVDD), U12.20 (VDD)
- net BUTTON: now also SW1.D
- net CAP_MIS: now also U9.51 (PA10); no longer U9.65 (PB5)
- net ENC_A: now also R37.2, SW1.A
- net ENC_B: now also R38.2, SW1.B
- net FAULT_IN: now also U9.49 (PB15); no longer U9.63 (PB3)
- net GND: now also Q1.3 (S), U13.1 (GND), U7.3 (CAT), Brd1.1 (GND), C19.2, C30.2, C33.2, C35.2, D3.2 (A), R22.2, SW1.6, SW1.7, SW1.C, SW1.E, U12.10 (GND), U12.15 (DGND), U12.16 (GND), U12.21 (GND)
- net HEATBED: now also R24.2
- net I2C_SCL: now also Brd1.3 (SCL)
- net I2C_SDA: now also Brd1.4 (SDA)
- net LED_BLUE: now also D7.1 (K)
- net LED_COOLING: now also D11.1 (K)
- net LED_GREEN: now also D6.1 (K)
- net LED_PD: now also D12.1 (K)
- net LED_PREHEAT: now also D8.1 (K)
- net LED_RED: now also D5.1 (K)
- net LED_REFLOW: now also D10.1 (K)
- net LED_SOAK: now also D9.1 (K)
- net PPHV: now also D2.1 (K), R21.1, U4.1
- net SINK_EN: now also U9.50 (PC6); no longer U9.64 (PB4)
- net at U7.1 (AN): now also R24.1
- net at U7.4 (EMI): now also Q1.1 (G), D3.1 (K), R22.1
- net at U7.6 (COL): now also R21.2
- net at U13.2 (T-): now also U11.2
- net at U13.3 (T+): now also U11.1
- net THERMO_SCK: now reaches U13.5 (SCK)
- net THERMO_CS: now reaches U13.6 (~{CS})
- net THERMO_MISO: now reaches U13.7 (SO)
- net at U9.43 (VLXSMPS): now also L3.1; no longer L2.1
- net at Q1.2 (D): now also D2.2 (A), U4.2
- net PT_CS: now reaches U9.19 (PA4)
- net PT_CS: now also U12.13 (~{CS})
- net PT_DRDY: now reaches U9.20 (PA5)
- net PT_DRDY: now also U12.18 (~{DRDY})
- net PT: no longer names the net of U9.12 (PC3)
- new net: D8.2 (A), R32.1
- new net: R39.1, U12.1 (BIAS), U12.2 (REFIN+)
- new net: R39.2, U12.3 (REFIN-), U12.4 (ISENSOR)
- new net: U12.5 (FORCE+), U12.6 (FORCE2), U14.1
- new net: C38.1, U12.7 (RTDIN+), U14.2
- new net: C38.2, U12.8 (RTDIN-), U12.9 (FORCE-), U14.3
- new net: D6.2 (A), R30.1
- new net: D10.2 (A), R34.1
- new net: D11.2 (A), R35.1
- new net: D9.2 (A), R33.1
- new net: L2.1, L3.2
- new net: D5.2 (A), R29.1
- new net: D12.2 (A), R36.1
- new net: D7.2 (A), R31.1
- new net PT_MISO: U12.14 (SDO), U9.64 (PB4)
- new net PT_MOSI: U12.11 (SDI), U9.65 (PB5)
- new net PT_SCK: U12.12 (SCLK), U9.63 (PB3)
- no-connect marks 7 -> 13
Other:
- note added: "100Ω RTD = 100nF 1kΩ RTD = 10nF"
- note added: "32MB FLASH"
- note added: "3V3 BUCK CONVERTER"
- note added: "BOARD TEMP SENSOR"
- note added: "BUZZER AND LEDS"
- note added: "CURRENT SENSOR"
- note added: "DECOUPLING"
- note added: "EMBER"
- note added: "EXTERNAL TEMPERATURE SENSORS"
- note added: "HEATBED CONTROL"
- note added: "I/O"
- note added: "NFC"
- note added: "PERIPHERALS"
- note added: "STM32"
- note added: "USB ESD"
- note added: "USB-C"
- note added: "USB-C PD"
- title: (none) -> Ember
- moved on the sheet: AE1, BUZZER1, C10, C11, C12, C13, C14, C16, C18, C20, C21, C22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
Changed lines of the file:
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@@
 	(generator_version "9.0")
 	(paper "A3")
+	(title_block
+		(title "Ember")
+	)

Commit message: finish schematic
Parts:
- added C42, C43: 330pF, Capacitor_SMD:C_0402_1005Metric, symbol Device:C
- C11, C13: footprint Capacitor_SMD:C_0603_1608Metric -> Capacitor_SMD:C_0402_1005Metric
- R1, R12, R4, R6: footprint Resistor_SMD:R_0603_1608Metric -> Resistor_SMD:R_0402_1005Metric
Connections:
- net CC1: now also C42.1
- net CC2: now also C43.1
- net GND: now also C42.2, C43.2

Commit message: stuff
Connections:
- net PPHV: now also R18.2, U5.8 (Vbus), U5.9 (Vin-); no longer U1.20 (PPHV)
- net PPHV_R: now reaches R18.1, U5.10 (Vin+)
- net PPHV_R: now also U1.20 (PPHV)

Commit message: start routing
Parts:
- C17: footprint Capacitor_SMD:C_0603_1608Metric -> Capacitor_SMD:C_0402_1005Metric
Connections:
- net PPHV: now also R18.1; no longer C2.1, C5.1, C8.1, R18.2
- net PPHV_R: now also C2.1, C5.1, C8.1, R18.2; no longer R18.1
Other:
- moved on the sheet: R18

Commit message: udpate routing
Parts:
- removed Q1: IRFB3207PBF, lcsc:TO-220-3_L10.0-W4.5-P2.54-T, symbol lcsc:IRFB3207PBF
- added Q3: IRF1018ESTRLPBF, lcsc:TO-263-3_L10.2-W10.7-P5.08-LS16.2-BR, symbol lcsc:IRF1018ESTRLPBF
Connections:
- net GND: now also Q3.3 (S)
- net PT_DRDY: now also U9.25 (PC4); no longer U9.20 (PA5)
- net at D3.1 (K), R22.1, U7.4 (EMI): now also Q3.1 (G)
- net at U12.5 (FORCE+), U12.6 (FORCE2): now also U14.3; no longer U14.1
- net at C38.2, U12.8 (RTDIN-), U12.9 (FORCE-): now also U14.1; no longer U14.3
- net at D2.2 (A), U4.2: now also Q3.2 (D)
- net C_SBU1: no longer names the net of USB1.9 (SBU1)
- net C_SBU1: no longer U3.1 (C_SBU1)
- net C_SBU2: no longer names the net of USB1.3 (SBU2)
- net C_SBU2: no longer U3.2 (C_SBU2)
- no-connect marks 13 -> 16
