File: hardware/board/ember.kicad_sch (KiCad schematic)
At the start: 133 parts, among them Q2 2SC1815_C727146, Q3 IRF1018ESTRLPBF, SW1 EC11E18244A5, SW2 SW_Push, SW3 SW_Push, U1 TPS25730D, U10 NT3H2111W0FHKH, U11 DB128L-5.08-2P-BK-S, U12 MAX31865xTP, U13 MAX6675ISA+T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

Commit message: changed buck
Parts:
- removed C14: 120uF, Capacitor_SMD:CP_Elec_6.3x7.7, symbol Device:C_Polarized
- removed C3: 22uF, Capacitor_SMD:CP_Elec_6.3x5.4, symbol Device:C_Polarized
- removed D1: SS56, lcsc:SMA_L4.3-W2.6-LS5.2-RD, symbol lcsc:SS56
- removed L1: FXL0650-8R2-M, lcsc:IND-SMD_L7.0-W6.6_FXL0650, symbol lcsc:FXL0650-8R2-M
- removed U2: LM22676MR-ADJ, Package_SO:TI_SO-PowerPAD-8, symbol Regulator_Switching:LM22676MR-ADJ
- added C14: 100nF, Capacitor_SMD:C_0402_1005Metric, symbol Device:C
- added C3: 10uF, Capacitor_SMD:C_0805_2012Metric, symbol Device:C
- added C44, C45: 22uF, Capacitor_SMD:C_0805_2012Metric, symbol Device:C
- added L1: FXL0530-4R7-M, lcsc:IND-SMD_L5.4-W5.2_FXL0530, symbol lcsc:FXL0530-4R7-M
- added U15: TPS56339DDC, Package_TO_SOT_SMD:SOT-23-6, symbol Regulator_Switching:TPS56339DDC
- C12: value 10nF -> 100nF; footprint Capacitor_SMD:C_0402_1005Metric -> Capacitor_SMD:C_0603_1608Metric
- C6: value 6.8uF -> 10uF; footprint Capacitor_SMD:C_0603_1608Metric -> Capacitor_SMD:C_0805_2012Metric
- R15: value 976 -> 30.9K
- R17: value 1.54K -> 10K
- R5: value 470K -> 30; footprint Resistor_SMD:R_0603_1608Metric -> Resistor_SMD:R_0402_1005Metric
Connections:
- net +3.3V: now also R15.1, C44.1, C45.1, L1.1; no longer R17.1
- net GND: now also C12.2, R17.2, C3.2, C44.2, C45.2, U15.1 (GND); no longer R15.2
- net PPHV: now also C12.1, C3.1, U15.3 (VIN); no longer R5.1
- net at R5.2: now also C14.1
- new net: R5.1, U15.6 (BOOT)
- new net: C14.2, L1.2, U15.2 (SW)
- new net: R15.2, R17.1, U15.4 (FB)
- no-connect marks 16 -> 17
Other:
- moved on the sheet: C6

Commit message: udpate pcb with fixes
Parts:
- removed Q3: IRF1018ESTRLPBF, lcsc:TO-263-3_L10.2-W10.7-P5.08-LS16.2-BR, symbol lcsc:IRF1018ESTRLPBF
- removed R21: 1K, Resistor_SMD:R_0402_1005Metric, symbol Device:R
- removed U7: TLP183(GRH-TPL,E(T, lcsc:SOIC-4_L3.6-W4.4-P2.54-LS7.0-TL, symbol lcsc:TLP183(GRH-TPL,E(T
- added C46: 4.7uF, Capacitor_SMD:C_0603_1608Metric, symbol Device:C
- added C47: 100nF, Capacitor_SMD:C_0603_1608Metric, symbol Device:C
- added H4: MountingHole, MountingHole:MountingHole_2.2mm_M2, symbol Mechanical:MountingHole
- added Q1: IRFS7440TRLPBF, lcsc:TO-263-2_L10.0-W9.1-P5.08-LS15.2-BR, symbol lcsc:IRFS7440TRLPBF
- added U2: TC4431EOA, lcsc:SOIC-8_L4.9-W3.9-P1.27-LS6.0-BL, symbol lcsc:TC4431EOA
Connections:
- net GND: now also C46.2, C47.2, Q1.3 (S), U2.3 (~{LOCK_DIS}), U2.4 (GND), U2.5 (GND)
- net PPHV: now also C46.1, C47.1, U2.1 (VDD), U2.8 (VDD)
- net at R24.1: now also U2.2 (IN)
- net at D3.1 (K), R22.1: now also Q1.1 (G), U2.6 (~{OUT}), U2.7 (~{OUT})
- net at D2.2 (A), U4.2: now also Q1.4 (D)
Other:
- moved on the sheet: D2, D3, R22, R24, U4

Commit message: finish board and prod/case files
Parts:
- R1: LCSC (none) -> C3013157
- R12, R4: LCSC (none) -> C2998070
- R13: LCSC (none) -> C96273
- R2: LCSC (none) -> C2998174
- R3: LCSC (none) -> C852970
- R39: footprint Resistor_SMD:R_0402_1005Metric -> Resistor_SMD:R_0805_2012Metric; LCSC (none) -> C153298
- R7: LCSC (none) -> C852750
Changed lines of the file:
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@@
 			)
 		)
+		(property "LCSC" "C96273"
+			(at 83.82 212.09 0)
+			(effects
+				(font
+					(size 1.27 1.27)
+				)
+				(hide yes)
+			)
+		)
 		(pin "1"
 		)
@@
 			)
 		)
+		(property "LCSC" "C852970"
+			(at 43.18 201.93 0)
+			(effects
+				(font
+					(size 1.27 1.27)
+				)
+				(hide yes)
+			)
+		)
 		(pin "1"
 		)
@@
 			)
 		)
-		(property "Footprint" "Resistor_SMD:R_0402_1005Metric"
+		(property "Footprint" "Resistor_SMD:R_0805_2012Metric"
 			(at 368.808 215.9 90)
 			(effects
@@
 			)
 		)
+		(property "LCSC" "C153298"
+			(at 367.03 215.9 0)
+			(effects
+				(font
+					(size 1.27 1.27)
+				)
+				(hide yes)
+			)
+		)
 		(pin "1"
 		)
@@
 			)
 		)
+		(property "LCSC" "C852750"
+			(at 63.5 212.09 0)
+			(effects
+				(font
+					(size 1.27 1.27)
+				)
+				(hide yes)
+			)
+		)
 		(pin "1"
 		)
@@
 			)
 		)
+		(property "LCSC" "C2998174"
+			(at 20.32 212.09 0)
+			(effects
+				(font
+					(size 1.27 1.27)
+				)
+				(hide yes)
+			)
+		)
 		(pin "1"
 		)
@@
 			)
 		)
+		(property "LCSC" "C2998070"
+			(at 83.82 201.93 0)
+			(effects
+				(font
+					(size 1.27 1.27)
+				)
+				(hide yes)
+			)
+		)
 		(pin "1"
 		)
@@
 			)
 		)
+		(property "LCSC" "C2998070"
+			(at 43.18 212.09 0)
+			(effects
+				(font
+					(size 1.27 1.27)
+				)
+				(hide yes)
+			)
+		)
 		(pin "1"
 		)
@@
 			(at 20.32 201.93 0)
 			(effects
+				(font
+					(size 1.27 1.27)
+				)
+				(hide yes)
+			)
+		)
+		(property "LCSC" "C3013157"
+			(at 20.32 201.93 0)
+			(effects

Commit message: fixed via sizing
Parts:
- D10, D11, D8, D9: LCSC (none) -> C965800
- D12: LCSC (none) -> C2290
- D5: LCSC (none) -> C965799
- D6: LCSC (none) -> C19171301
- D7: LCSC (none) -> C965807
Changed lines of the file:
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@@
 			)
 		)
+		(property "LCSC" "C965800"
+			(at 279.4 171.45 0)
+			(effects
+				(font
+					(size 1.27 1.27)
+				)
+				(hide yes)
+			)
+		)
 		(pin "1"
 		)
@@
 		(on_board yes)
 		(dnp no)
-		(fields_autoplaced yes)
 		(property "Reference" "U12"
 			(at 347.5833 203.2 0)
@@
 			)
 		)
-		(property "Sim.Pins" "1=K 2=A"
+		(property "LCSC" "C965800"
 			(at 279.4 184.15 0)
 			(effects
@@
 			)
 		)
-		(property "Sim.Pins" "1=K 2=A"
+		(property "LCSC" "C965800"
 			(at 279.4 190.5 0)
 			(effects
@@
 			)
 		)
-		(property "Sim.Pins" "1=K 2=A"
+		(property "LCSC" "C965800"
 			(at 279.4 177.8 0)
 			(effects
@@
 			)
 		)
+		(property "LCSC" "C19171301"
+			(at 279.4 158.75 0)
+			(effects
+				(font
+					(size 1.27 1.27)
+				)
+				(hide yes)
+			)
+		)
 		(pin "1"
 		)
@@
 			)
 		)
+		(property "LCSC" "C965807"
+			(at 279.4 165.1 0)
+			(effects
+				(font
+					(size 1.27 1.27)
+				)
+				(hide yes)
+			)
+		)
 		(pin "1"
 		)
@@
 			)
 		)
-		(property "Sim.Pins" "1=K 2=A"
+		(property "LCSC" "C2290"
 			(at 279.4 196.85 0)
 			(effects
@@
 			(at 279.4 152.4 0)
 			(effects
+				(font
+					(size 1.27 1.27)
+				)
+				(hide yes)
+			)
+		)
+		(property "LCSC" "C965799"
+			(at 279.4 152.4 0)
+			(effects

Commit message: added speaker stuff and usb c pd driver
Other:
- note added: "I2C ADDRESS: 0x20"
- note added: "Value: 0"
- note added: "Value: 1"
- note added: "Value: 3"
- note added: "Value: 7"
Changed lines of the file:
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@@
+		)
+	)
+	(text "Value: 7"
+		(exclude_from_sim no)
+		(at 48.768 226.06 0)
+		(effects
+			(font
+				(size 1.27 1.27)
+			)
+		)
+	)
+	(text "Value: 1"
+		(exclude_from_sim no)
+		(at 90.678 225.552 0)
+		(effects
+			(font
+				(size 1.27 1.27)
+			)
 		)
 	)
@@
 		)
 	)
+	(text "Value: 0"
+		(exclude_from_sim no)
+		(at 24.892 225.806 0)
+		(effects
+			(font
+				(size 1.27 1.27)
+			)
+		)
+	)
+	(text "I2C ADDRESS: 0x20"
+		(exclude_from_sim no)
+		(at 99.568 129.032 0)
+		(effects
+			(font
+				(size 1.27 1.27)
+			)
+		)
+	)
 	(text "STM32"
 		(exclude_from_sim no)
@@
 			)
 		)
+	)
+	(text "Value: 3"
+		(exclude_from_sim no)
+		(at 70.358 225.806 0)
+		(effects
+			(font
+				(size 1.27 1.27)
+			)
+		)

Commit message: nfc stuff
Connections:
- net +3.3V: now also C16.1, U5.6 (VS)
Other:
- note added: "ADDRESS: 0x40"
- note added: "ADDRESS: 1001000x"
Changed lines of the file:
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@@
 		)
 	)
+	(text "ADDRESS: 0x40"
+		(exclude_from_sim no)
+		(at 152.4 126.746 0)
+		(effects
+			(font
+				(size 1.27 1.27)
+			)
+		)
+	)
 	(text "3V3 BUCK CONVERTER"
 		(exclude_from_sim no)
@@
 		)
 	)
+	(text "ADDRESS: 1001000x"
+		(exclude_from_sim no)
+		(at 182.88 247.396 0)
+		(effects
+			(font
+				(size 1.27 1.27)
+			)
+		)
+	)
 	(text "HEATBED CONTROL"
 		(exclude_from_sim no)
@@
 	)
 	(junction
+		(at 133.35 99.06)
+		(diameter 0)
+		(color 0 0 0 0)
+	)
+	(junction
 		(at 73.66 36.83)
 		(diameter 0)
@@
 	(wire
 		(pts
+			(xy 133.35 97.79) (xy 133.35 99.06)
+		)
+		(stroke
+			(width 0)
+			(type default)
+		)
+	)
+	(wire
+		(pts
 			(xy 259.08 265.43) (xy 259.08 267.97)
 		)
@@
 	)
 	(symbol
+		(lib_id "power:+3.3V")
+		(at 133.35 97.79 0)
+		(unit 1)
+		(exclude_from_sim no)
+		(in_bom yes)
+		(on_board yes)
+		(dnp no)
+		(property "Reference" "#PWR0103"
+			(at 133.35 101.6 0)
+			(effects
+				(font
+					(size 1.27 1.27)
+				)
+				(hide yes)
+			)
+		)
+		(property "Value" "+3.3V"
+			(at 133.35 93.726 0)
+			(effects
+				(font
+					(size 1.27 1.27)
+				)
+			)
+		)
+		(property "Footprint" ""
+			(at 133.35 97.79 0)
+			(effects
+				(font
+					(size 1.27 1.27)
+				)
+				(hide yes)
+			)
+		)
+		(property "Datasheet" ""
+			(at 133.35 97.79 0)
+			(effects
+				(font
+					(size 1.27 1.27)
+				)
+				(hide yes)
+			)
+		)
+		(property "Description" "Power symbol creates a global label with name \"+3.3V\""
+			(at 133.35 97.79 0)
+			(effects
+				(font
+					(size 1.27 1.27)
+				)
+				(hide yes)
+			)
+		)
+		(pin "1"
+		)
+		(instances
+			(project "ember"
+				(path "/8a6c6108-ba3a-4119-97a5-40ac844b74e3"
+					(reference "#PWR0103")
+					(unit 1)
+				)
+			)
+		)
+	)
+	(symbol
 		(lib_id "Sensor_Temperature:MAX31865xTP")
 		(at 342.9 226.06 0)
@@
 				)
 				(justify left)
-				(hide yes)
 			)
 		)
@@
 				)
 				(justify left)
-				(hide yes)
 			)
 		)

Commit message: update code and flx haeter
Parts:
- added U7: MAX6682MUA+, lcsc:MSOP-8_L3.0-W3.0-P0.65-LS4.9-BL, symbol lcsc:MAX6682MUA+
Changed lines of the file:
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@@
+	)
+	(symbol
+		(lib_id "lcsc:MAX6682MUA+")
+		(at 387.35 196.85 0)
+		(unit 1)
+		(exclude_from_sim no)
+		(in_bom yes)
+		(on_board yes)
+		(dnp no)
+		(fields_autoplaced yes)
+		(property "Reference" "U7"
+			(at 387.35 185.42 0)
+			(effects
+				(font
+					(size 1.27 1.27)
+				)
+			)
+		)
+		(property "Value" "MAX6682MUA+"
+			(at 387.35 187.96 0)
+			(effects
+				(font
+					(size 1.27 1.27)
+				)
+			)
+		)
+		(property "Footprint" "lcsc:MSOP-8_L3.0-W3.0-P0.65-LS4.9-BL"
+			(at 387.35 208.28 0)
+			(effects
+				(font
+					(size 1.27 1.27)
+				)
+				(hide yes)
+			)
+		)
+		(property "Datasheet" "https://lcsc.com/product-detail/Temperature-Sensors_MAXIM_MAX6682MUA_MAX6682MUA_C143562.html"
+			(at 387.35 210.82 0)
+			(effects
+				(font
+					(size 1.27 1.27)
+				)
+				(hide yes)
+			)
+		)
+		(property "Description" ""
+			(at 387.35 196.85 0)
+			(effects
+				(font
+					(size 1.27 1.27)
+				)
+				(hide yes)
+			)
+		)
+		(property "LCSC Part" "C143562"
+			(at 387.35 213.36 0)
+			(effects
+				(font
+					(size 1.27 1.27)
+				)
+				(hide yes)
+			)
+		)
+		(pin "2"
+		)
+		(pin "1"
+		)
+		(pin "4"
+		)
+		(pin "6"
+		)
+		(pin "8"
+		)
+		(pin "5"
+		)
+		(pin "3"
+		)
+		(pin "7"
+		)
+		(instances
+			(project ""
+				(path "/8a6c6108-ba3a-4119-97a5-40ac844b74e3"
+					(reference "U7")
+					(unit 1)
+				)
+			)
+		)
 	)
 	(symbol
