File: hardware/board/ember.kicad_pcb (KiCad board)
At the start: 4 copper layers, 128 parts, among them Q1 IRFB3207PBF, Q2 2SC1815_C727146, SW1 EC11E18244A5, SW2 SW_Push, SW3 SW_Push, U1 TPS25730D, U10 NT3H2111W0FHKH, U11 DB128L-5.08-2P-BK-S, U12 MAX31865xTP, U13 MAX6675ISA+T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

Commit message: finish schematic
Parts:
- added C42: 330pF, Capacitor_SMD:C_0402_1005Metric, F.Cu at (63.9, 67.8)
- added C43: 330pF, Capacitor_SMD:C_0402_1005Metric, F.Cu at (62.0, 67.8)
- C11, C13: footprint Capacitor_SMD:C_0603_1608Metric -> Capacitor_SMD:C_0402_1005Metric
- R1, R12, R4, R6: footprint Resistor_SMD:R_0603_1608Metric -> Resistor_SMD:R_0402_1005Metric
- moved USB1 224.0 mm to (51.3, 55.7), turned to -90 degrees
- moved C10 200.6 mm to (57.5, 68.7)
- moved C15 200.4 mm to (62.3, 52.9)
- moved C17 200.4 mm to (59.2, 58.3)
- moved R20 200.4 mm to (57.7, 58.2)
- moved U3 200.4 mm to (62.3, 56.4)
- moved C13 199.8 mm to (57.0, 73.0), turned to 180 degrees
- moved C4 199.7 mm to (67.1, 68.3)
- moved C7 199.7 mm to (67.1, 69.9)
- moved C8 199.7 mm to (66.5, 77.4)
- moved C9 199.7 mm to (67.1, 71.5)
- moved R1 199.7 mm to (55.1, 72.2)
- moved R10 199.7 mm to (60.0, 69.0)
- moved R12 199.7 mm to (50.9, 72.2)
- moved R13 199.7 mm to (50.9, 74.8)
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Routing:
- net LDO_3V3: track 17.4 -> 0.00 mm, vias 3 -> 0
- net /ADCIN4: track 10.1 -> 0.00 mm, vias 2 -> 0
- net /ADCIN3: track 8.00 -> 0.00 mm, vias 2 -> 0
- net /ADCIN2: track 6.61 -> 0.00 mm, vias 2 -> 0
- net GND: track 5.11 -> 0.00 mm
- net /ADCIN1: track 3.92 -> 0.00 mm
- net /DRAIN: track 2.74 -> 0.00 mm
- net +3.3V: track 2.43 -> 0.00 mm
- net LDO_1V5: track 1.76 -> 0.00 mm
- net Net-(R8-Pad2): track 1.44 -> 0.00 mm
- net Net-(R10-Pad2): track 1.29 -> 0.00 mm
- net /FAULT_IN: track 1.24 -> 0.00 mm
- net Net-(R9-Pad2): track 1.14 -> 0.00 mm
Other:
- board outline added: 150 x 50 mm

Commit message: stuff
Parts:
- moved C16 156.3 mm to (170.2, 24.2)
- moved R18 156.3 mm to (174.8, 22.3)
- moved R23 156.3 mm to (161.9, 22.9)
- moved U5 156.3 mm to (166.2, 23.4)
- moved R13 148.6 mm to (194.5, 36.6), turned to 90 degrees
- moved R12 147.3 mm to (194.5, 39.3), turned to 90 degrees
- moved R7 145.6 mm to (193.0, 36.8), turned to 90 degrees
- moved R6 144.2 mm to (192.9, 39.3), turned to 90 degrees
- moved R4 143.3 mm to (191.7, 36.2), turned to 90 degrees
- moved USB1 142.8 mm to (194.1, 55.7), turned to 90 degrees
- moved R3 142.0 mm to (191.6, 38.7), turned to 90 degrees
- moved R2 140.6 mm to (190.4, 36.8), turned to 90 degrees
- moved R1 139.2 mm to (190.4, 39.3), turned to 90 degrees
- moved C13 135.9 mm to (188.4, 38.4), turned to 0 degrees
- moved R16 134.2 mm to (186.6, 35.3), turned to 180 degrees
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Connections:
- R18 pad 1: Net-(U5-Vin+) -> PPHV_R
- R18 pad 2: Net-(U5-Vbus) -> PPHV
- U1 pad 20: PPHV -> PPHV_R
- U5 pad 10: Net-(U5-Vin+) -> PPHV_R
- U5 pad 8: Net-(U5-Vbus) -> PPHV
- U5 pad 9: Net-(U5-Vbus) -> PPHV
Routing:
- added copper zone on F.Cu, net VBUS

Commit message: start routing
Parts:
- C17: footprint Capacitor_SMD:C_0603_1608Metric -> Capacitor_SMD:C_0402_1005Metric
- moved U14 177.2 mm to (141.9, 25.5)
- moved C38 162.2 mm to (141.1, 32.7), turned to 180 degrees
- moved R19 159.5 mm to (82.9, 42.6)
- moved C19 159.5 mm to (78.2, 42.6)
- moved U6 159.5 mm to (80.4, 42.1)
- moved R39 155.5 mm to (145.1, 37.1), turned to 90 degrees
- moved U12 154.5 mm to (141.1, 36.6), turned to 180 degrees
- moved C20 153.9 mm to (57.7, 56.9)
- moved U8 153.9 mm to (63.4, 54.5)
- moved C33 152.8 mm to (125.5, 32.7)
- moved U11 152.8 mm to (128.3, 25.4)
- moved U13 152.8 mm to (127.8, 37.3)
- moved U4 147.7 mm to (117.1, 25.4), turned to 0 degrees
- moved C35 147.7 mm to (143.2, 40.6), turned to 0 degrees
- moved C30 146.2 mm to (141.7, 41.0), turned to -90 degrees
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Connections:
- C2 pad 1: PPHV -> PPHV_R
- C5 pad 1: PPHV -> PPHV_R
- C8 pad 1: PPHV -> PPHV_R
- R18 pad 1: PPHV_R -> PPHV
- R18 pad 2: PPHV -> PPHV_R
Routing:
- net /C_CC2: track 0.00 -> 14.5 mm, vias 0 -> 2
- net /DN: track 0.00 -> 2.88 mm
- net /DP: track 0.00 -> 2.51 mm
- net /C_SBU1: track 0.00 -> 0.76 mm, vias 0 -> 1

Commit message: udpate routing
Parts:
- removed Q1: IRFB3207PBF, lcsc:TO-220-3_L10.0-W4.5-P2.54-T
- added Q3: IRF1018ESTRLPBF, lcsc:TO-263-3_L10.2-W10.7-P5.08-LS16.2-BR, F.Cu at (104.0, 34.7)
- moved D10 63.4 mm to (129.0, 80.4)
- moved D11 63.4 mm to (131.6, 80.4)
- moved D12 63.4 mm to (134.2, 80.4)
- moved D5 63.4 mm to (116.1, 80.4)
- moved R30 63.4 mm to (120.4, 76.9)
- moved R31 63.4 mm to (122.4, 76.9)
- moved R33 63.4 mm to (126.4, 76.9)
- moved R34 63.4 mm to (128.4, 76.9)
- moved D7 63.4 mm to (121.3, 80.4)
- moved D8 63.4 mm to (123.9, 80.4)
- moved D9 63.4 mm to (126.5, 80.4)
- moved R29 63.4 mm to (118.4, 76.9)
- moved R32 63.4 mm to (124.4, 76.9)
- moved R36 63.4 mm to (134.0, 77.1)
- moved D6 63.4 mm to (118.7, 80.4)
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Connections:
- U14 pad 1: Net-(U12-FORCE+) -> Net-(U12-FORCE-)
- U14 pad 3: Net-(U12-FORCE-) -> Net-(U12-FORCE+)
- U3 pad 1: /C_SBU1 -> unconnected-(U3-C_SBU1-Pad1)
- U3 pad 2: /C_SBU2 -> unconnected-(U3-C_SBU2-Pad2)
- U9 pad 20: /PT_DRDY -> unconnected-(U9-PA5-Pad20)
- U9 pad 25: unconnected-(U9-PC4-Pad25) -> /PT_DRDY
- USB1 pad 3: /C_SBU2 -> unconnected-(USB1-SBU2-Pad3)
- USB1 pad 9: /C_SBU1 -> unconnected-(USB1-SBU1-Pad9)
Routing:
- net /I2C_SDA: track 0.00 -> 145.7 mm, vias 0 -> 3
- net /I2C_SCL: track 0.00 -> 143.8 mm, vias 0 -> 3
- net /FIELD_DETECT: track 0.00 -> 121.8 mm, vias 0 -> 2
- net /THERMO_MISO: track 0.00 -> 112.3 mm
- net /THERMO_CS: track 0.00 -> 108.4 mm
- net /THERMO_SCK: track 0.00 -> 107.5 mm
- net /BUTTON: track 0.00 -> 106.0 mm, vias 0 -> 2
- net /ENC_B: track 0.00 -> 103.1 mm, vias 0 -> 1
- net /ENC_A: track 0.00 -> 93.5 mm, vias 0 -> 1
- net /PT_DRDY: track 0.00 -> 91.3 mm, vias 0 -> 2
- net /PT_CS: track 0.00 -> 84.9 mm, vias 0 -> 2
- net /HEATBED: track 0.00 -> 71.6 mm, vias 0 -> 2
- net /PT_MISO: track 0.00 -> 67.9 mm
- net /PT_MOSI: track 0.00 -> 67.6 mm
- net /PT_SCK: track 0.00 -> 67.1 mm, vias 0 -> 2
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- added copper zone on F.Cu, net +3.3V
- added copper zone on In2.Cu, net +3.3V
- added copper zone on B.Cu, net GND
- added copper zone on F.Cu, net GND
- added copper zone on In1.Cu, net GND
- added copper zone on F.Cu, net PPHV
- added copper zone on F.Cu, net PPHV_R
Other:
- outline, holes or cut-outs redrawn
- board text added: "@NotARoomba"
- board text added: "EMBER"

Commit message: finished PCB
Parts:
- added H1: MountingHole, MountingHole:MountingHole_2.2mm_M2, F.Cu at (206.9, 111.1)
- added H2: MountingHole, MountingHole:MountingHole_2.2mm_M2, F.Cu at (206.9, 67.6)
- added H3: MountingHole, MountingHole:MountingHole_2.2mm_M2, F.Cu at (129.5, 111.1)
- TP1, TP2, TP3: moved to B.Cu
- moved TP2 113.5 mm to (120.4, 96.5), turned to 90 degrees
- moved TP1 111.2 mm to (124.6, 96.5), turned to 90 degrees
- moved TP3 110.2 mm to (122.5, 96.5)
- moved C20 68.1 mm to (103.9, 104.2), turned to 0 degrees
- moved FL1 67.8 mm to (112.8, 108.6), turned to 45 degrees
- moved U8 60.3 mm to (101.5, 98.9), turned to 180 degrees
- moved Brd1 57.4 mm to (161.2, 89.8)
- moved C34 57.4 mm to (121.6, 99.8), turned to 0 degrees
- moved C5 57.3 mm to (101.2, 70.4)
- moved C2 57.3 mm to (99.0, 70.4)
- moved C8 57.3 mm to (102.7, 70.4)
- moved C23 57.1 mm to (110.5, 100.1)
- moved AE1 57.0 mm to (91.0, 111.8)
- moved BUZZER1 56.9 mm to (141.9, 98.2)
- moved C24 56.9 mm to (120.8, 106.3)
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Connections:
- U8 pad 9: unconnected-(U8-EP-Pad9) -> GND
Routing:
- net /LED_PD: track 0.00 -> 62.8 mm
- net /FAULT_IN: track 7.20 -> 64.8 mm
- net /SINK_EN: track 7.69 -> 63.9 mm
- net /LED_SOAK: track 0.00 -> 49.8 mm
- net /LED_PREHEAT: track 0.00 -> 49.2 mm
- net /CAP_MIS: track 10.1 -> 57.0 mm
- net /DP: track 2.51 -> 47.2 mm, vias 0 -> 3
- net /DN: track 2.54 -> 45.5 mm, vias 0 -> 3
- net /LED_COOLING: track 0.00 -> 36.7 mm
- net /LED_REFLOW: track 0.00 -> 36.0 mm
- net /BUZZER: track 0.00 -> 30.5 mm, vias 0 -> 2
- net +3.3V: track 49.6 -> 80.0 mm, vias 41 -> 65
- net /LED_BLUE: track 0.00 -> 25.0 mm, vias 0 -> 2
- net /LED_GREEN: track 0.00 -> 24.8 mm, vias 0 -> 2
- net /LED_RED: track 0.00 -> 24.7 mm, vias 0 -> 2
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- added copper zone on B.Cu, net PPHV
- added copper zone on In1.Cu, net PPHV
- added copper zone on In2.Cu, net PPHV
Other:
- board text added: "+"
- board text added: "-"
- board text added: "BOOT"
- board text added: "COOL"
- board text added: "ERROR"
- board text added: "GOOD"
- board text added: "HOTPLATE"
- board text added: "PD"
- board text added: "PREHEAT"
- board text added: "REFLOW"
- board text added: "RESET"
- board text added: "RTD"
- board text added: "SOAK"
- board text added: "STATUS"
- board text added: "THERMOCOUPLE"
- board text added: "V1"
