File: hardware/board/ember.kicad_pcb (KiCad board)
At the start: 4 copper layers, 150 x 50 mm, 133 parts, among them Q2 2SC1815_C727146, Q3 IRF1018ESTRLPBF, SW1 EC11E18244A5, SW2 SW_Push, SW3 SW_Push, U1 TPS25730D, U10 NT3H2111W0FHKH, U11 DB128L-5.08-2P-BK-S, U12 MAX31865xTP, U13 MAX6675ISA+T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

Commit message: changed buck
Parts:
- removed D1: SS56, lcsc:SMA_L4.3-W2.6-LS5.2-RD
- removed U2: LM22676MR-ADJ, Package_SO:TI_SO-PowerPAD-8
- added C44: 22uF, Capacitor_SMD:C_0805_2012Metric, F.Cu at (123.8, 79.8)
- added C45: 22uF, Capacitor_SMD:C_0805_2012Metric, F.Cu at (126.1, 79.8)
- added U15: TPS56339DDC, Package_TO_SOT_SMD:SOT-23-6, F.Cu at (112.9, 82.0)
- C12: value 10nF -> 100nF; footprint Capacitor_SMD:C_0402_1005Metric -> Capacitor_SMD:C_0603_1608Metric
- C14: value 120uF -> 100nF; footprint Capacitor_SMD:CP_Elec_6.3x7.7 -> Capacitor_SMD:C_0402_1005Metric
- C3: value 22uF -> 10uF; footprint Capacitor_SMD:CP_Elec_6.3x5.4 -> Capacitor_SMD:C_0805_2012Metric
- C6: value 6.8uF -> 10uF; footprint Capacitor_SMD:C_0603_1608Metric -> Capacitor_SMD:C_0805_2012Metric
- L1: value FXL0650-8R2-M -> FXL0530-4R7-M; footprint lcsc:IND-SMD_L7.0-W6.6_FXL0650 -> lcsc:IND-SMD_L5.4-W5.2_FXL0530
- R15: value 976 -> 30.9K
- R17: value 1.54K -> 10K
- R5: value 470K -> 30; footprint Resistor_SMD:R_0603_1608Metric -> Resistor_SMD:R_0402_1005Metric
- moved C14 15.4 mm to (112.8, 84.7)
- moved R5 15.2 mm to (111.8, 84.7), turned to -90 degrees
- moved R15 14.5 mm to (109.8, 81.0), turned to 0 degrees
- moved R17 12.7 mm to (111.2, 79.5)
- moved C6 9.86 mm to (113.1, 77.4), turned to 180 degrees
- moved C19 9.33 mm to (122.7, 72.6)
- moved R19 9.33 mm to (118.0, 72.7)
- moved U6 9.33 mm to (120.5, 73.1)
- moved L1 6.13 mm to (118.4, 82.0)
- moved C3 4.26 mm to (113.1, 75.3), turned to 180 degrees
- moved C12 3.02 mm to (113.2, 79.3)
Connections:
- C12 pad 1: Net-(U2-BOOT) -> PPHV
- C12 pad 2: Net-(D1-K) -> GND
- C14 pad 1: +3.3V -> Net-(C14-Pad1)
- C14 pad 2: GND -> Net-(U15-SW)
- L1 pad 1: Net-(D1-K) -> +3.3V
- L1 pad 2: +3.3V -> Net-(U15-SW)
- R15 pad 1: Net-(U2-FB) -> +3.3V
- R15 pad 2: GND -> Net-(U15-FB)
- R17 pad 1: +3.3V -> Net-(U15-FB)
- R17 pad 2: Net-(U2-FB) -> GND
- R5 pad 1: PPHV -> Net-(U15-BOOT)
- R5 pad 2: Net-(U2-EN) -> Net-(C14-Pad1)
- U8 pad 9: GND -> unconnected-(U8-EP-Pad9)
Routing:
- net Net-(D1-K): track 15.8 -> 0.00 mm
- net +3.3V: track 80.0 -> 70.9 mm
- net Net-(U15-SW): track 0.00 -> 5.46 mm
- net Net-(U2-FB): track 5.04 -> 0.00 mm
- net /TEMP_ALERT: track 51.5 -> 47.0 mm
- net PPHV: track 14.9 -> 10.8 mm, vias 190 -> 0
- net /HEATBED: track 71.3 -> 75.3 mm
- net /I2C_SCL: track 144.8 -> 148.8 mm
- net /I2C_SDA: track 146.4 -> 150.3 mm
- net Net-(U15-FB): track 0.00 -> 2.70 mm
- net Net-(U2-EN): track 2.61 -> 0.00 mm
- net Net-(U2-BOOT): track 1.35 -> 0.00 mm
- net Net-(U15-BOOT): track 0.00 -> 1.26 mm
- net Net-(C14-Pad1): track 0.00 -> 1.06 mm
- net GND: vias 740 -> 151

Commit message: different buck and heatbed
Parts:
- moved Q3 5.02 mm to (135.3, 78.5)
- moved C45 4.78 mm to (123.8, 84.0), turned to 0 degrees
- moved C44 1.90 mm to (123.8, 81.8), turned to 0 degrees
- renumbered TP3 to GND, TP2 to SWCLK, TP1 to SWDIO
Connections:
- U8 pad 9: unconnected-(U8-EP-Pad9) -> GND
Routing:
- net Net-(D3-K): track 9.68 -> 14.0 mm
- net Net-(D2-A): track 47.0 -> 45.2 mm
- net +3.3V: track 70.9 -> 71.4 mm, vias 65 -> 66
- net PPHV: vias 0 -> 191
- net GND: vias 151 -> 1180
